File: RTDTemp.kicad_pcb (KiCad board)
At the start: 2 copper layers, 80 x 100 mm, 109 parts, among them J1 Conn_01x02, J2 Conn_01x02, J3 Car Power, J4 CAN_In, J5 CAN_Out, SW1 SW_Push, U1 Nucleo_L432KC, U2 PWR_REG_PQMC3-Dx-Sx-S, U3 ADM3055E, U4 CDSOT23-T24CAN

Commit message: savestate
Other:
- rule pad_to_mask_clearance: 0.2 -> 0
